Commit message: modification for compiling

File: src/microEpsilon_scanControl/description/urdf/scanCONTROL_2600-100_macro.urdf.xacro (robot description, xacro)
@@ -24,12 +24,13 @@
             </collision>
         </link>
-        <!--<joint name="${prefix}scanner_laser_joint" type="fixed">
+        <!--joint name="${prefix}scanner_laser_joint" type="fixed">
             <origin xyz="0 0 0" rpy="0 0 ${pi}" />
             <parent link="${prefix}scanner_link"/>
             <child link="${prefix}scanner_laser_link" />
-        </joint>-->
+        </joint-->
         <joint name="${prefix}scanner_laser_joint" type="fixed">
             <origin xyz="0.0383464 0.109996 0.135064" rpy="${radians(0.242595)} ${radians(0.0646638)} ${radians(-92.129)}" />
-            <parent link="tool0"/>
+            <!--parent link="tool0"/-->
+            <parent link="${prefix}scanner_link"/>
             <child link="${prefix}scanner_laser_link" />
         </joint>
