Commit message: successfully compile and run microepsilon!

File: src/microEpsilon_scanControl/description/urdf/scanCONTROL_2600-100.urdf.xacro (robot description, xacro)
@@ -6,5 +6,7 @@
 <!-- sensor -->
   <xacro:scanCONTROL_2600-100 prefix="scanCONTROL_2600-100" parent="base_link">
-      <origin xyz="0 0 0" rpy="0 0 0" />
+      <!-- <origin xyz="0 0 0" rpy="0 0 0" /> -->
+      <!-- <origin xyz="0.0383464 0.109996 0.135064" rpy="${radians(0)} ${radians(0)} ${radians(180)}" /> -->
+      <origin xyz="0.0383464 0.109996 0.135064" rpy="${radians(0)} ${radians(180)} ${radians(180)}" />
   </xacro:scanCONTROL_2600-100>
 </robot>

File: src/microEpsilon_scanControl/description/urdf/scanCONTROL_2600-100_macro.urdf.xacro (robot description, xacro)
@@ -24,15 +24,16 @@
             </collision>
         </link>
-        <!--joint name="${prefix}scanner_laser_joint" type="fixed">
-            <origin xyz="0 0 0" rpy="0 0 ${pi}" />
-            <parent link="${prefix}scanner_link"/>
-            <child link="${prefix}scanner_laser_link" />
-        </joint-->
         <joint name="${prefix}scanner_laser_joint" type="fixed">
-            <origin xyz="0.0383464 0.109996 0.135064" rpy="${radians(0.242595)} ${radians(0.0646638)} ${radians(-92.129)}" />
-            <!--parent link="tool0"/-->
+            <!-- <origin xyz="0 0 0" rpy="0 0 ${pi}" /> -->
+            <origin xyz="0 0 0" rpy="${radians(90)} ${radians(0)} ${radians(0)}" />
             <parent link="${prefix}scanner_link"/>
             <child link="${prefix}scanner_laser_link" />
         </joint>
+        <!-- <joint name="${prefix}scanner_laser_joint" type="fixed"> -->
+            <!-- <origin xyz="0.0383464 0.109996 0.135064" rpy="${radians(0.242595)} ${radians(0.0646638)} ${radians(-92.129)}" /> -->
+            <!--parent link="tool0"/-->
+            <!-- <parent link="${prefix}scanner_link"/> -->
+            <!-- <child link="${prefix}scanner_laser_link" /> -->
+        <!-- </joint>  -->
         <link name="${prefix}scanner_laser_link" />
   </xacro:macro>
