Commit message: Succussfully compile and run robviz file

File: src/RT_monitoring_application/scanning_workcell/urdf/workcell.xacro (robot description, xacro)
@@ -3,5 +3,6 @@
   <property name="pi" value="3.141592654" />
   <xacro:property name="tcp_frame">
-    <origin xyz="0.24646 -0.02439 0.433932" rpy="${pi} -1.047197555 ${pi}" />
+    <!--origin xyz="0.24646 -0.02439 0.433932" rpy="${pi} -1.047197555 ${pi}" /-->
+    <origin xyz="0.002785 0.271833 0.174487" rpy="-${pi} 0.0 -${pi}" />
   </xacro:property>
   <xacro:property name="workobject_frame">

Commit message: add microepsilon workcell with robot scanning cell

File: src/RT_monitoring_application/scanning_workcell/urdf/workcell.xacro (robot description, xacro)
@@ -26,5 +26,5 @@
     <parent link="tool0"/>
     <child link="head0"/>
-    <origin xyz="0 0 0" rpy="0 0 ${pi/2}" />
+    <origin xyz="0 0 0" rpy="${radians(20)} 0 ${radians(90)}" />
     <axis xyz="0 0 1"/>
   </joint>
