Commit message: change microepsilon URDF to make the point cloud in correct orientation and position. Add microepsilon scanning video

File: src/RT_monitoring_application/scanning_workcell/urdf/head.xacro (robot description, xacro)
@@ -4,5 +4,6 @@
     <visual>
       <geometry>
-        <mesh filename="package://scanning_workcell/meshes/head/visual/head_wt03.stl" />
+        <!-- <mesh filename="package://scanning_workcell/meshes/head/visual/head_wt03.stl" /> -->
+        <mesh filename="package://scanning_workcell/meshes/head/visual/laserhead.stl" />
       </geometry>
       <material name="dark_gray">
@@ -12,5 +13,5 @@
     <collision>
       <geometry>
-        <mesh filename="package://scanning_workcell/meshes/head/collision/head_wt03.stl" />
+        <mesh filename="package://scanning_workcell/meshes/head/collision/laserhead.stl" />
       </geometry>
       <material name="yellow">

File: src/microEpsilon_scanControl/microepsilon_workcell/urdf/scanCONTROL_2900-50_macro.urdf.xacro (robot description, xacro)
@@ -25,5 +25,5 @@
     </link>
     <joint name="${prefix}scanner_laser_joint" type="fixed">
-        <origin xyz="0 0 0" rpy="${radians(0)} ${radians(90)} ${radians(180)}" />
+        <origin xyz="0 0 0" rpy="${radians(0)} ${radians(0)} ${radians(180)}" />
         <parent link="${prefix}scanner_link"/>
         <child link="${prefix}scanner_laser_link" />

File: src/microEpsilon_scanControl/microepsilon_workcell/urdf/workcell.xacro (robot description, xacro)
@@ -12,5 +12,5 @@
   <!-- sensor -->
   <xacro:scanCONTROL_2900-50 prefix="scanCONTROL_2900-50_" parent="link_6">
-    <origin xyz="0.1 0.2 -0.1" rpy="${radians(180)} ${radians(-90)} ${radians(-90)}" />
+    <origin xyz="0.1 0.2 -0.1" rpy="${radians(0)} ${radians(0)} ${radians(90)}" />
   </xacro:scanCONTROL_2900-50>
 </robot>

Commit message: change error in multi-planner segmentation

File: src/RT_monitoring_application/scanning_workcell/urdf/head.xacro (robot description, xacro)
@@ -5,5 +5,5 @@
       <geometry>
         <!-- <mesh filename="package://scanning_workcell/meshes/head/visual/head_wt03.stl" /> -->
-        <mesh filename="package://scanning_workcell/meshes/head/visual/laserhead.stl" />
+        <mesh filename="package://scanning_workcell/meshes/head/visual/laserhead.STL" />
       </geometry>
       <material name="dark_gray">
@@ -13,5 +13,5 @@
     <collision>
       <geometry>
-        <mesh filename="package://scanning_workcell/meshes/head/collision/laserhead.stl" />
+        <mesh filename="package://scanning_workcell/meshes/head/collision/laserhead.STL" />
       </geometry>
       <material name="yellow">
