Commit message: modify some code for point cloud processing with microepsilon

File: src/microEpsilon_scanControl/microepsilon_workcell/urdf/scanCONTROL_2900-50_macro.urdf.xacro (robot description, xacro)
@@ -25,5 +25,5 @@
     </link>
     <joint name="${prefix}scanner_laser_joint" type="fixed">
-        <origin xyz="0 0 0" rpy="${radians(0)} ${radians(180)} ${radians(180)}" />
+        <origin xyz="0 0 0" rpy="${radians(0)} ${radians(90)} ${radians(180)}" />
         <parent link="${prefix}scanner_link"/>
         <child link="${prefix}scanner_laser_link" />

File: src/microEpsilon_scanControl/microepsilon_workcell/urdf/workcell.xacro (robot description, xacro)
@@ -11,6 +11,6 @@
   <xacro:include filename="$(find microepsilon_workcell)/urdf/scanCONTROL_2900-50_macro.urdf.xacro" />
   <!-- sensor -->
-  <xacro:scanCONTROL_2900-50 prefix="scanCONTROL_2900-50_" parent="tcp0">
-    <origin xyz="0.0383464 0.109996 0.135064" rpy="${radians(0)} ${radians(90)} ${radians(-90)}" />
+  <xacro:scanCONTROL_2900-50 prefix="scanCONTROL_2900-50_" parent="link_6">
+    <origin xyz="0.1 0.2 -0.1" rpy="${radians(180)} ${radians(-90)} ${radians(-90)}" />
   </xacro:scanCONTROL_2900-50>
 </robot>
