Commit message: Major update for June
- Successfully connected the micorepsilon sensor
- Upload programs for acceleration-velocity-power control
- upload experiment data for control
- make some minor changes for program naming

File: src/microEpsilon_scanControl/microepsilon_workcell/urdf/workcell.xacro (robot description, xacro)
@@ -11,6 +11,6 @@
   <xacro:include filename="$(find microepsilon_workcell)/urdf/scanCONTROL_2900-50_macro.urdf.xacro" />
   <!-- sensor -->
-  <xacro:scanCONTROL_2900-50 prefix="scanCONTROL_2900-50_" parent="link_6">
-    <origin xyz="0.1 0.2 -0.1" rpy="${radians(0)} ${radians(0)} ${radians(90)}" />
+  <xacro:scanCONTROL_2900-50 prefix="scanCONTROL_2900-50_" parent="tool0">
+    <origin xyz="0.10135 0.2 0.15" rpy="${radians(-90)} ${radians(0)} ${radians(90)}" />
   </xacro:scanCONTROL_2900-50>
 </robot>
