Commit message: successfully test all functions for height monitoring

File: src/microEpsilon_scanControl/microepsilon_workcell/urdf/workcell_kuka.xacro (robot description, xacro)
@@ -2,6 +2,6 @@
 <robot name="microepsilon_workcell" xmlns:xacro="http://ros.org/wiki/xacro">
   <!-- Robot cell with working head and camera-->
-  <xacro:include filename="$(find scanning_workcell)/urdf/workcell_kuka.xacro"/>
-  <joint name="scanning_workcell" type="fixed">
+  <xacro:include filename="$(find simtech_kuka_workcell)/urdf/workcell.xacro"/>
+  <joint name="simtech_kuka_workcell" type="fixed">
     <parent link="world"/>
     <child link="base_link"/>
@@ -11,6 +11,8 @@
   <xacro:include filename="$(find microepsilon_workcell)/urdf/scanCONTROL_2900-50_macro.urdf.xacro" />
   <!-- sensor -->
-  <xacro:scanCONTROL_2900-50 prefix="scanCONTROL_2900-50_" parent="tool0">
-    <origin xyz="0.10135 0.2 0.15" rpy="${radians(-90)} ${radians(0)} ${radians(90)}" />
+  <xacro:scanCONTROL_2900-50 prefix="scanCONTROL_2900-50_" parent="tcp_link">
+    <!-- relative to the tool0 (6 axix/flange) -->
+    <!-- <origin xyz="0.10135 0.2 0.15" rpy="${radians(-90)} ${radians(0)} ${radians(90)}" />  -->
+    <origin xyz="0 -0.2 -0.15" rpy="${radians(90)} ${radians(180)} 0" />
   </xacro:scanCONTROL_2900-50>
 </robot>

File: src/simtech_kuka/simtech_kuka_workcell/urdf/kuka_robot.xacro (robot description, xacro)
@@ -3,5 +3,5 @@
     <property name="pi" value="3.141592654"/>
     <!-- Robot -->
-    <xacro:include filename="$(find simtech_kuka_workcell)/urdf/kr120r2500pro_macro.xacro"/>
+    <xacro:include filename="$(find simtech_kuka_robot_support)/urdf/kr120r2500pro_macro.xacro"/>
     <xacro:kuka_kr120r2500pro prefix=""/>
     <joint name="kr120r2500pro" type="fixed">

File: src/simtech_kuka/simtech_kuka_workcell/urdf/kuka_robot_B.xacro (robot description, xacro)
@@ -3,5 +3,5 @@
     <property name="pi" value="3.141592654"/>
     <!-- Robot -->
-    <xacro:include filename="$(find simtech_kuka_workcell)/urdf/kr120r2500proB_macro.xacro"/>
+    <xacro:include filename="$(find simtech_kuka_robot_support)/urdf/kr120r2500proB_macro.xacro"/>
     <xacro:kuka_kr120r2500proB prefix=""/>
     <joint name="kr120r2500proB" type="fixed">

File: src/simtech_kuka/simtech_kuka_workcell/urdf/kuka_robot_simulation.xacro (robot description, xacro)
@@ -3,5 +3,5 @@
     <property name="pi" value="3.141592654"/>
     <!-- Robot -->
-    <xacro:include filename="$(find simtech_kuka_workcell)/urdf/kr120r2500pro_macro.xacro"/>
+    <xacro:include filename="$(find simtech_kuka_robot_support)/urdf/kr120r2500pro_macro.xacro"/>
     <xacro:kuka_kr120r2500pro prefix=""/>
     <joint name="kr120r2500pro" type="fixed">

File: src/simtech_kuka/simtech_kuka_workcell/urdf/workcell.xacro (robot description, xacro)
@@ -1,12 +1,48 @@
 <?xml version="1.0" ?>
 <robot name="simtech_kuka_workcell" xmlns:xacro="http://ros.org/wiki/xacro">
-    <property name="pi" value="3.141592654"/>
-    <link name="world"/>
-    <!-- Robot -->
-    <xacro:include filename="$(find simtech_kuka_workcell)/urdf/kuka_robot.xacro"/>
-    <joint name="kuka_robot" type="fixed">
-        <parent link="world"/>
-        <child link="base_link"/>
-        <origin xyz="0 0 0.067" rpy="0 0 0"/>
-    </joint>
+  <property name="pi" value="3.141592654" />
+  <link name="world"/>
+  <xacro:property name="tcp_frame">
+    <!-- from data sheet -->
+    <origin xyz="-0.0109374151 -0.25882666 0.286677063" rpy="0 0.0 -${pi/2}" />
+  </xacro:property>
+  <xacro:property name="workobject_frame">
+      <!-- from datasheet -->
+    <!-- <origin xyz="1.14256 -1.59023279 0.0157544041" rpy="0 0 0" /> -->
+    <origin xyz="1.3 0 0.4157544041" rpy="0 0 0" />
+  </xacro:property>
+  <!-- Robot -->
+  <xacro:include filename="$(find simtech_kuka_workcell)/urdf/kuka_robot.xacro"/>
+  <joint name="kuka_robot" type="fixed">
+      <parent link="world"/>
+      <child link="base_link"/>
+      <origin xyz="0 0 0.0" rpy="0 0 0"/>
+  </joint>
+  <!-- Head -->
+  <xacro:include filename="$(find simtech_kuka_workcell)/urdf/head.xacro"/>
+  <joint name="laser_head" type="fixed">
+    <parent link="tool0"/>
+    <child link="laser_head_link"/>
+    <!-- <origin xyz="0.14633243 -0.083423 0.172" rpy="${radians(0)} ${radians(180)} 0" /> -->
+    <origin xyz="-0.14633243 0.083423 0.172" rpy="${radians(0)} ${radians(180)} ${radians(180)}" />
+    <!-- <origin xyz="0.14633243 -0.083423 0.172" rpy="${radians(0)} ${radians(0)} 0" /> -->
+    <axis xyz="0 0 1"/>
+  </joint>
+  <!-- TCP -->
+  <!-- tool0 is $FLANGE in KUKA KRC controllers. -->
+  <link name="tcp_link"/>
+  <joint name="tcp_joint" type="fixed">
+    <parent link="tool0"/>
+    <child link="tcp_link"/>
+    <xacro:insert_block name="tcp_frame" />
+    <axis xyz="0 0 1"/>
+  </joint>
+  <!-- Workobject -->
+  <link name="workobject" />
+  <joint name="workobject" type="fixed">
+    <parent link="base_link" />
+    <child link="workobject" />
+    <xacro:insert_block name="workobject_frame" />
+    <!--<axis xyz="0 0 1"/>-->
+  </joint>
 </robot>

File: src/simtech_kuka/simtech_kuka_workcell/urdf/workcell_test.xacro (robot description, xacro)
@@ -3,7 +3,7 @@
     <property name="pi" value="3.141592654"/>
     <link name="world"/>
-    <!-- Robot -->
-    <xacro:include filename="$(find simtech_kuka_workcell)/urdf/kuka_robot_simulation.xacro"/>
-    <joint name="kuka_robot" type="fixed">
+    <!-- Robot (with table) -->
+    <xacro:include filename="$(find simtech_kuka_workcell)/urdf/workcell.xacro"/>
+    <joint name="workcell" type="fixed">
         <parent link="world"/>
         <child link="base_link"/>

Commit message: Update code (successful software demo for height monitoring)

File: src/microEpsilon_scanControl/microepsilon_workcell/urdf/workcell_kuka.xacro (robot description, xacro)
@@ -14,5 +14,5 @@
     <!-- relative to the tool0 (6 axix/flange) -->
     <!-- <origin xyz="0.10135 0.2 0.15" rpy="${radians(-90)} ${radians(0)} ${radians(90)}" />  -->
-    <origin xyz="0 -0.2 -0.15" rpy="${radians(90)} ${radians(180)} 0" />
+    <origin xyz="0 -0.2 -0.15" rpy="${radians(90)} ${radians(180)} ${radians(180)}" />
   </xacro:scanCONTROL_2900-50>
 </robot>
