Commit message: Update the correct laser head urdf file

File: src/simtech_robot_laser_control/urdf/head.xacro (robot description, xacro)
@@ -4,13 +4,15 @@
     <visual>
       <geometry>
-        <mesh filename="package://simtech_robot_laser_control/meshes/head/visual/head_wt03.stl" />
+        <!-- <mesh filename="package://scanning_workcell/meshes/head/visual/head_wt03.stl" /> -->
+        <mesh filename="package://scanning_workcell/meshes/head/visual/laserhead.STL" scale = "0.001 0.001 0.001"/>
       </geometry>
       <material name="dark_gray">
-        <color rgba="0.3 0.4 0.3 1"/>
+        <!-- <color rgba="0.3 0.4 0.3 1"/> -->
+        <color rgba="${175/255} ${175/255} ${169/255} 1.0"/>
       </material>
     </visual>
     <collision>
       <geometry>
-        <mesh filename="package://simtech_robot_laser_control/meshes/head/collision/head_wt03.stl" />
+        <mesh filename="package://scanning_workcell/meshes/head/collision/laserhead.STL" scale = "0.001 0.001 0.001"/>
       </geometry>
       <material name="yellow">

File: src/simtech_robot_laser_control/urdf/workcell.xacro (robot description, xacro)
@@ -27,6 +27,5 @@
     <parent link="tool0"/>
     <child link="head0"/>
-    <origin xyz="0 0 0" rpy="0 0 ${pi/2}" />
-    <!--origin xyz="0 0 0" rpy="0 0 0" /-->
+    <origin xyz="0.14633243 -0.083423 0.172" rpy="${radians(0)} ${radians(180)} 0" />
     <axis xyz="0 0 1"/>
   </joint>
