Commit message: Updata code for data fusion, minor changes to the height monitoring program on max min calculation

File: src/simtech_kuka/simtech_kuka_workcell/urdf/workcell.xacro (robot description, xacro)
@@ -11,4 +11,8 @@
     <!-- <origin xyz="1.14256 -1.59023279 0.0157544041" rpy="0 0 0" /> -->
     <origin xyz="1.3 0 0.4157544041" rpy="0 0 0" />
+  </xacro:property>
+  <xacro:property name="camera_frame">
+    <!-- origin xyz="0.2879 -0.0399 0.1267" rpy="1.55420 0.00225 1.59185" /-->
+    <origin xyz="0.2328 0.181 -0.0168" rpy="0.0016279188408910522 -0.009261168793408879 -0.05185504283900785" />
   </xacro:property>
   <!-- Robot -->
@@ -46,3 +50,10 @@
     <!--<axis xyz="0 0 1"/>-->
   </joint>
+   <!-- Camera -->
+   <link name="camera0" />
+   <joint name="tool0-camera0" type="fixed">
+     <parent link="tool0"/>
+     <child link="camera0"/>
+     <xacro:insert_block name="camera_frame" />
+   </joint>
 </robot>
