Commit message: update robot model

File: src/simtech_kuka/simtech_kuka_kr90_support/urdf/kr90r2700.xacro (robot description, xacro)
@@ -1,5 +1,5 @@
 <?xml version="1.0"?>
 <robot name="kuka_kr90r2700" xmlns:xacro="http://wiki.ros.org/xacro">
-  <xacro:include filename="$(find kuka_kr90_support)/urdf/kr90r2700_macro.xacro" />
+  <xacro:include filename="$(find simtech_kuka_kr90_support)/urdf/kr90r2700_macro.xacro" />
   <xacro:kuka_kr90r2700 prefix=""/>
 </robot>

File: src/simtech_kuka/simtech_kuka_kr90_support/urdf/kr90r2700_macro.xacro (robot description, xacro)
@@ -8,5 +8,5 @@
         <origin xyz="0 0 0" rpy="0 0 0"/>
         <geometry>
-          <mesh scale="0.001 0.001 0.001" filename="package://kuka_kr90_support/meshes/kr90r2700/visual/base_link.stl" />
+          <mesh scale="0.001 0.001 0.001" filename="package://simtech_kuka_kr90_support/meshes/kr90r2700/visual/base_link.stl" />
         </geometry>
         <xacro:material_kuka_pedestal />
@@ -15,5 +15,5 @@
         <origin xyz="0 0 0" rpy="0 0 0"/>
         <geometry>
-          <mesh scale="0.001 0.001 0.001" filename="package://kuka_kr90_support/meshes/kr90r2700/collision/base_link.stl" />
+          <mesh scale="0.001 0.001 0.001" filename="package://simtech_kuka_kr90_support/meshes/kr90r2700/collision/base_link.stl" />
         </geometry>
       </collision>
@@ -23,5 +23,5 @@
         <origin xyz="0 0 0" rpy="0 0 0"/>
         <geometry>
-          <mesh scale="0.001 0.001 0.001" filename="package://kuka_kr90_support/meshes/kr90r2700/visual/link_1.stl" />
+          <mesh scale="0.001 0.001 0.001" filename="package://simtech_kuka_kr90_support/meshes/kr90r2700/visual/link_1.stl" />
         </geometry>
         <xacro:material_kuka_orange />
@@ -30,5 +30,5 @@
         <origin xyz="0 0 0" rpy="0 0 0"/>
         <geometry>
-          <mesh scale="0.001 0.001 0.001" filename="package://kuka_kr90_support/meshes/kr90r2700/collision/link_1.stl" />
+          <mesh scale="0.001 0.001 0.001" filename="package://simtech_kuka_kr90_support/meshes/kr90r2700/collision/link_1.stl" />
         </geometry>
       </collision>
@@ -38,5 +38,5 @@
         <origin xyz="0 0 0" rpy="0 0 0"/>
         <geometry>
-          <mesh scale="0.001 0.001 0.001" filename="package://kuka_kr90_support/meshes/kr90r2700/visual/link_2.stl"/>
+          <mesh scale="0.001 0.001 0.001" filename="package://simtech_kuka_kr90_support/meshes/kr90r2700/visual/link_2.stl"/>
         </geometry>
         <xacro:material_kuka_orange />
@@ -45,5 +45,5 @@
         <origin xyz="0 0 0" rpy="0 0 0"/>
         <geometry>
-          <mesh scale="0.001 0.001 0.001" filename="package://kuka_kr90_support/meshes/kr90r2700/collision/link_2.stl" />
+          <mesh scale="0.001 0.001 0.001" filename="package://simtech_kuka_kr90_support/meshes/kr90r2700/collision/link_2.stl" />
         </geometry>
       </collision>
@@ -53,5 +53,5 @@
         <origin xyz="0 0 0" rpy="0 0 0"/>
         <geometry>
-          <mesh scale="1 1 1" filename="package://kuka_kr90_support/meshes/kr90r2700/visual/link_3.stl" />
+          <mesh scale="1 1 1" filename="package://simtech_kuka_kr90_support/meshes/kr90r2700/visual/link_3.stl" />
         </geometry>
         <xacro:material_kuka_orange />
@@ -60,5 +60,5 @@
         <origin xyz="0 0 0" rpy="0 0 0"/>
         <geometry>
-          <mesh scale="0.001 0.001 0.001" filename="package://kuka_kr90_support/meshes/kr90r2700/collision/link_3.stl" />
+          <mesh scale="0.001 0.001 0.001" filename="package://simtech_kuka_kr90_support/meshes/kr90r2700/collision/link_3.stl" />
         </geometry>
       </collision>
@@ -68,5 +68,5 @@
         <origin xyz="0 0 0" rpy="0 0 0"/>
         <geometry>
-          <mesh scale="0.001 0.001 0.001" filename="package://kuka_kr90_support/meshes/kr90r2700/visual/link_4.stl" />
+          <mesh scale="0.001 0.001 0.001" filename="package://simtech_kuka_kr90_support/meshes/kr90r2700/visual/link_4.stl" />
         </geometry>
         <xacro:material_kuka_orange />
@@ -75,5 +75,5 @@
         <origin xyz="0 0 0" rpy="0 0 0"/>
         <geometry>
-          <mesh scale="0.001 0.001 0.001" filename="package://kuka_kr90_support/meshes/kr90r2700/collision/link_4.stl" />
+          <mesh scale="0.001 0.001 0.001" filename="package://simtech_kuka_kr90_support/meshes/kr90r2700/collision/link_4.stl" />
         </geometry>
       </collision>
@@ -83,5 +83,5 @@
         <origin xyz="0 0 0" rpy="0 0 0"/>
         <geometry>
-          <mesh scale="0.001 0.001 0.001" filename="package://kuka_kr90_support/meshes/kr90r2700/visual/link_5.stl" />
+          <mesh scale="0.001 0.001 0.001" filename="package://simtech_kuka_kr90_support/meshes/kr90r2700/visual/link_5.stl" />
         </geometry>
         <xacro:material_kuka_orange />
@@ -90,5 +90,5 @@
         <origin xyz="0 0 0" rpy="0 0 0"/>
         <geometry>
-          <mesh scale="0.001 0.001 0.001" filename="package://kuka_kr90_support/meshes/kr90r2700/collision/link_5.stl" />
+          <mesh scale="0.001 0.001 0.001" filename="package://simtech_kuka_kr90_support/meshes/kr90r2700/collision/link_5.stl" />
         </geometry>
       </collision>
@@ -98,5 +98,5 @@
         <origin xyz="0 0 0" rpy="0 0 0"/>
         <geometry>
-          <mesh scale="0.001 0.001 0.001" filename="package://kuka_kr90_support/meshes/kr90r2700/visual/link_6.stl" />
+          <mesh scale="0.001 0.001 0.001" filename="package://simtech_kuka_kr90_support/meshes/kr90r2700/visual/link_6.stl" />
         </geometry>
         <xacro:material_kuka_pedestal />
@@ -105,5 +105,5 @@
         <origin xyz="0 0 0" rpy="0 0 0"/>
         <geometry>
-          <mesh scale="0.001 0.001 0.001" filename="package://kuka_kr90_support/meshes/kr90r2700/collision/link_6.stl" />
+          <mesh scale="0.001 0.001 0.001" filename="package://simtech_kuka_kr90_support/meshes/kr90r2700/collision/link_6.stl" />
         </geometry>
       </collision>
