Commit message: Update code for microepsilon robviz

File: src/scanning_application/scanning_workcell/urdf/workcell.xacro (robot description, xacro)
@@ -4,5 +4,8 @@
   <xacro:property name="tcp_frame">
     <!--origin xyz="0.24646 -0.02439 0.433932" rpy="${pi} -1.047197555 ${pi}" /-->
-    <origin xyz="0.002785 0.271833 0.174487" rpy="-${pi} 0.0 -${pi}" />
+    <!-- SIMTech Valleyblock setting -->
+    <!-- <origin xyz="0.002785 0.271833 0.174487" rpy="-${pi} 0.0 -${pi}" /> -->
+    <!-- CT2B setting Quaternion: [ 0.1311496, 0, -0.9913626, 0 ]-->
+    <origin xyz="0.031965 0.001138 0.557156" rpy="0 -0.2630569 3.1415927" />
   </xacro:property>
   <xacro:property name="workobject_frame">
