Commit message: Update ABB robot table

File: src/simtech_abb/simtech_workcell/urdf/workcell.xacro (robot description, xacro)
@@ -8,5 +8,13 @@
         <parent link="world"/>
         <child link="base_link"/>
-        <origin xyz="0 0 0.067" rpy="0 0 0"/>
+        <origin xyz="0 0 0" rpy="0 0 0"/>
+    </joint>
+    <!-- Robot table -->
+    <xacro:include filename="$(find simtech_workcell)/urdf/irbp_a750.xacro"/>
+    <joint name="irbp_a750" type="fixed">
+        <parent link="world"/>
+        <child link="irbp_a750/base_link"/>
+        <!-- <origin xyz="1.753 0.015 -0.003" rpy="-0.005599 -0.005742 1.550718"/> -->
+        <origin xyz="-0.0625 -1.49743 -0.012" rpy="-0.005599 -0.005742 1.550718"/>
     </joint>
 </robot>
