Commit message: Update the ABB table

File: src/simtech_abb/simtech_workcell/urdf/irbp_a750.xacro (robot description, xacro)
@@ -84,5 +84,5 @@
     <parent link="${name}base_link" />
     <child link="${name}link_1" />
-    <origin rpy="0 0 0" xyz="0 0 0" />
+    <origin rpy="0 0 0" xyz="0 0.1 0" />
     <axis xyz="0 0 1" />
   </joint>
@@ -90,5 +90,5 @@
     <parent link="${name}link_1" />
     <child link="${name}link_2" />
-    <origin rpy="0 0 0" xyz="0 0 1.020" />
+    <origin rpy="0 0 0" xyz="0 0.04 0.4" />
     <axis xyz="1 0 0" />
     <limit effort="100" lower="-3.1590" upper="3.1590" velocity="2.6180" />
@@ -97,5 +97,5 @@
     <parent link="${name}link_2" />
     <child link="${name}link_3" />
-    <origin rpy="0 0 0" xyz="0 0 0" />
+    <origin rpy="0 0 0" xyz="0.01 0.01 0" />
     <axis xyz="0 1 0" />
   </joint>
@@ -103,5 +103,5 @@
     <parent link="${name}link_3" />
     <child link="${name}link_4" />
-    <origin rpy="0 0 0" xyz="0 0 -0.120" />
+    <origin rpy="0 0 0" xyz="0 0 0.43" />
     <axis xyz="0 0 1" />
     <limit effort="100" velocity="3.1416" />
@@ -112,3 +112,20 @@
     <origin rpy="0 0 0" xyz="0 0 0" />
   </joint>
+  <!-- Table -->
+    <link name="table0">
+        <visual>
+            <geometry>
+                <mesh filename="package://simtech_workcell/meshes/table/table.stl"/>
+            </geometry>
+            <material name="gray">
+                <color rgba="0.4 0.4 0.4 0.8"/>
+            </material>
+        </visual>
+    </link>
+    <joint name="table0" type="fixed">
+        <parent link="irbp_a750/tool0"/>
+        <child link="table0"/>
+        <origin xyz="0 0 0" rpy="0 0 0"/>
+        <axis xyz="0 0 1"/>
+    </joint>
 </robot>

File: src/simtech_abb/simtech_workcell/urdf/workcell.xacro (robot description, xacro)
@@ -16,5 +16,7 @@
         <child link="irbp_a750/base_link"/>
         <!-- <origin xyz="1.753 0.015 -0.003" rpy="-0.005599 -0.005742 1.550718"/> -->
-        <origin xyz="-0.0625 -1.49743 -0.012" rpy="-0.005599 -0.005742 1.550718"/>
+        <!-- Works for ABB 250 -->
+        <!-- <origin xyz="-0.0625 -1.49743 -0.012" rpy="-0.005599 -0.005742 1.550718"/> -->
+        <origin xyz="-0.3625 -1.49743 -0.012" rpy="-0.005599 -0.005742 -1.550718"/>
     </joint>
 </robot>
